Commit message: feat: complete workspace restructuring, exclude build artifacts, refactor URDF and optimize Gazebo simulation

File: src/limo_gazebo_sim/urdf/limo_ackerman.xacro (robot description, xacro)
@@ -2,10 +2,9 @@
 <robot name="limo_ackerman" xmlns:xacro="http://ros.org/wiki/xacro">
     <xacro:arg name="robot_namespace" default="/" />
-    <xacro:include filename="$(find limo_gazebo_sim)/urdf/limo_xacro.xacro" />
-    <xacro:include filename="$(find limo_gazebo_sim)/urdf/limo_steering_hinge.xacro" />
-    <xacro:include filename="$(find limo_gazebo_sim)/urdf/limo_ackerman.gazebo" />
-    <!-- Variables -->
+    <!-- 导入解耦后的传感器与执行机构模块 -->
+    <xacro:include filename="$(find limo_gazebo_sim)/urdf/sensors.xacro" />
+    <xacro:include filename="$(find limo_gazebo_sim)/urdf/actuators.xacro" />
+    <!-- ================= 几何与物理参数定义 ================= -->
     <xacro:property name="M_PI" value="3.14159"/>
-    <!-- Vehicle Geometries -->
     <xacro:property name="base_x_size" value="0.26" />
     <xacro:property name="base_y_size" value="0.24" />
@@ -17,23 +16,24 @@
     <xacro:property name="wheel_length" value="0.09" />
     <xacro:property name="wheel_radius" value="0.09" />
+    <xacro:property name="wheel_scale" value="2 2 2" />
+    <!-- ================= 底盘基准与车身 Link ================= -->
     <link name="base_footprint"/>
     <joint name="base_joint" type="fixed">
-    <parent link="base_footprint"/>
-    <child link="base_link"/>
-    <origin xyz="0.0 0.0 0.30" rpy="0 0 0"/>
+        <parent link="base_footprint"/>
+        <child link="base_link"/>
+        <origin xyz="0.0 0.0 0.30" rpy="0 0 0"/>
     </joint>
-    <!-- Base link -->
     <link name="base_link">
         <visual>
             <origin xyz="0 0 -0.30" rpy="0 0 1.57" />
             <geometry>
-                <mesh filename="package://limo_gazebo_sim/meshes/limo_base.dae" scale="2 2 2"/>
+                <mesh filename="package://limo_gazebo_sim/CAD/limo-model/limo_base.dae" scale="2 2 2"/>
             </geometry>
         </visual>
         <collision>
             <origin xyz="0 0 0" rpy="0 0 0" />
-          <geometry>
-              <box size="${base_x_size} ${base_y_size} ${base_z_size}"/>
-          </geometry>
+            <geometry>
+                <box size="${base_x_size} ${base_y_size} ${base_z_size}"/>
+            </geometry>
         </collision>
     </link>
@@ -52,4 +52,5 @@
         <child link="inertial_link" />
     </joint>
+    <!-- ================= 传感器装配 (包含 Gazebo 插件) ================= -->
     <xacro:limo_laser parent_prefix="base_link" frame_prefix="laser">
         <origin xyz="0.206 0 -0.068" rpy="0 0 0"/>
@@ -61,59 +62,67 @@
         <origin xyz="0.0 0 -0.2" rpy="0 0 0"/>
     </xacro:limo_imu>
-    <xacro:limo_left_steering_hinge parent_prefix="base_link" wheel_prefix="left_steering_hinge">
-        <origin xyz="${wheelbase/2} ${track/2} ${wheel_vertical_offset}" rpy="0 0  0" />
-    </xacro:limo_left_steering_hinge>
-    <xacro:limo_right_steering_hinge parent_prefix="base_link" wheel_prefix="right_steering_hinge">
+    <!-- ================= 前轮转向机构装配 (转向铰链节 + 前轮) ================= -->
+    <!-- 左前转向节及前轮 -->
+    <xacro:limo_steering_hinge parent_prefix="base_link" hinge_prefix="left_steering_hinge" wheel_prefix="front_left" reflect="1">
+        <origin xyz="${wheelbase/2} ${track/2} ${wheel_vertical_offset}" rpy="0 0 0" />
+    </xacro:limo_steering_hinge>
+    <!-- 右前转向节及前轮 -->
+    <xacro:limo_steering_hinge parent_prefix="base_link" hinge_prefix="right_steering_hinge" wheel_prefix="front_right" reflect="-1">
         <origin xyz="${wheelbase/2} ${-track/2} ${wheel_vertical_offset}" rpy="${M_PI} 0 0" />
-    </xacro:limo_right_steering_hinge>
-    <link name="rear_left_wheel_link">
-        <inertial>
-            <origin xyz="0 0 0" />
-            <mass value="0.5" />
-            <inertia ixx="0.01055" ixy="0" ixz="0" iyy="0.00075" iyz="0" izz="0.01055" />
-        </inertial>
-        <visual>
-            <origin xyz="0 0 0" rpy="0 0 0" />
-            <geometry>
-                <mesh filename="package://limo_gazebo_sim/meshes/limo_wheel.dae" scale="2 2 2" />
-            </geometry>
-        </visual>
-        <collision>
-            <origin xyz="0 ${wheel_length/2} 0" rpy="1.57 0 0" />
-          <geometry>
-              <cylinder length="${wheel_length}" radius="${wheel_radius}" />
-          </geometry>
-        </collision>
-    </link>
-    <joint name="rear_left_wheel" type="continuous">
-        <parent link="base_link"/>
-        <child link="rear_left_wheel_link"/>
+    </xacro:limo_steering_hinge>
+    <!-- ================= 后轮驱动轮装配 (复用通用轮系宏) ================= -->
+    <!-- 左后轮 -->
+    <xacro:limo_wheel parent_prefix="base_link" wheel_prefix="rear_left" reflect="1">
         <origin xyz="${-wheelbase/2} ${track/2} ${wheel_vertical_offset}" rpy="0 0 0" />
-        <axis xyz="0 1 0"/>
-    </joint>
-    <link name="rear_right_wheel_link">
-        <inertial>
-            <origin xyz="0 0 0" />
-            <mass value="0.5" />
-            <inertia ixx="0.01055" ixy="0" ixz="0" iyy="0.00075" iyz="0" izz="0.01055" />
-        </inertial>
-        <visual>
-            <origin xyz="0 0 0" rpy="0 0 0" />
-            <geometry>
-                <mesh filename="package://limo_gazebo_sim/meshes/limo_wheel.dae" scale="2 2 2" />
-            </geometry>
-        </visual>
-            <collision>
-                <origin xyz="0 ${wheel_length/2} 0" rpy="1.57 0 0" />
-              <geometry>
-                  <cylinder length="${wheel_length}" radius="${wheel_radius}" />
-              </geometry>
-            </collision>
-        </link>
-        <joint name="rear_right_wheel" type="continuous">
-            <parent link="base_link"/>
-            <child link="rear_right_wheel_link"/>
-            <origin xyz="${-wheelbase/2} ${-track/2} ${wheel_vertical_offset}" rpy="${M_PI} 0 0" />
-            <axis xyz="0 -1 0"/>
-        </joint>
+    </xacro:limo_wheel>
+    <!-- 右后轮 -->
+    <xacro:limo_wheel parent_prefix="base_link" wheel_prefix="rear_right" reflect="-1">
+        <origin xyz="${-wheelbase/2} ${-track/2} ${wheel_vertical_offset}" rpy="${M_PI} 0 0" />
+    </xacro:limo_wheel>
+    <!-- ================= Gazebo 仿真环境动力学与控制插件 ================= -->
+    <gazebo>
+        <mu1 value="10"/>
+        <mu2 value="10"/>
+        <kp value="10000000.0" />
+        <kd value="1.0" />
+        <fdir1 value="1 0 0"/>
+        <minDepth value="0.001" />
+        <maxContacts value="64"/>
+    </gazebo>
+    <gazebo>
+        <!-- ros_control 控制器插件 (提供转向节关节位置控制) -->
+        <plugin name="gazebo_ros_control" filename="libgazebo_ros_control.so">
+            <robotNamespace>$(arg robot_namespace)</robotNamespace>
+        </plugin>
+        <!-- 阿克曼转向运动学解算与驱动插件 -->
+        <plugin name="four_diff_controller" filename="libgazebo_ros_ackerman.so">
+            <updateRate>100.0</updateRate>
+            <robotNamespace>$(arg robot_namespace)</robotNamespace>
+            <leftFrontJoint>front_left_wheel</leftFrontJoint>
+            <rightFrontJoint>front_right_wheel</rightFrontJoint>
+            <leftRearJoint>rear_left_wheel</leftRearJoint>
+            <rightRearJoint>rear_right_wheel</rightRearJoint>
+            <leftHingeJoint>left_steering_hinge_wheel</leftHingeJoint>
+            <rightHingeJoint>right_steering_hinge_wheel</rightHingeJoint>
+            <wheelSeparation>0.344</wheelSeparation>
+            <wheelDiameter>0.18</wheelDiameter>
+            <wheelbase>${wheelbase}</wheelbase>
+            <wheelTrack>${track}</wheelTrack>
+            <robotBaseFrame>base_footprint</robotBaseFrame>
+            <commandTopic>cmd_vel</commandTopic>
+            <torque>50</torque>
+            <broadcastTF>true</broadcastTF>
+            <odometryTopic>odom</odometryTopic>
+            <odometryFrame>odom</odometryFrame>
+            <covariance_x>0.000100</covariance_x>
+            <covariance_y>0.000100</covariance_y>
+            <covariance_yaw>0.010000</covariance_yaw>
+        </plugin>
+        <!-- 关节状态发布插件 -->
+        <plugin name="joint_state_publisher" filename="libgazebo_ros_joint_state_publisher.so">
+            <jointName>front_left_wheel,front_right_wheel,rear_left_wheel,rear_right_wheel,left_steering_hinge_wheel,right_steering_hinge_wheel</jointName>
+            <updateRate>50.0</updateRate>
+            <robotNamespace>$(arg robot_namespace)</robotNamespace>
+        </plugin>
+    </gazebo>
 </robot>

File: src/limo_gazebo_sim/urdf/limo_four_diff.xacro (robot description, xacro)
@@ -2,9 +2,9 @@
 <robot name="limo_four_diff" xmlns:xacro="http://ros.org/wiki/xacro">
     <xacro:arg name="robot_namespace" default="/" />
-    <xacro:include filename="$(find limo_gazebo_sim)/urdf/limo_xacro.xacro" />
-    <xacro:include filename="$(find limo_gazebo_sim)/urdf/limo_four_diff.gazebo" />
-    <!-- Variables -->
+    <!-- 导入解耦后的传感器与执行机构模块 -->
+    <xacro:include filename="$(find limo_gazebo_sim)/urdf/sensors.xacro" />
+    <xacro:include filename="$(find limo_gazebo_sim)/urdf/actuators.xacro" />
+    <!-- ================= 几何与物理参数定义 ================= -->
     <xacro:property name="M_PI" value="3.14159"/>
-    <!-- Vehicle Geometries -->
     <xacro:property name="base_x_size" value="0.13" />
     <xacro:property name="base_y_size" value="0.12" />
@@ -16,24 +16,24 @@
     <xacro:property name="wheel_length" value="0.045" />
     <xacro:property name="wheel_radius" value="0.045" />
-  <link name="base_footprint"/>
-  <joint name="base_joint" type="fixed">
-    <parent link="base_footprint"/>
-    <child link="base_link"/>
-    <origin xyz="0.0 0.0 0.15" rpy="0 0 0"/>
-  </joint>
-    <!-- Base link -->
+    <xacro:property name="wheel_scale" value="2 2 2" />
+    <!-- ================= 底盘基准与车身 Link ================= -->
+    <link name="base_footprint"/>
+    <joint name="base_joint" type="fixed">
+        <parent link="base_footprint"/>
+        <child link="base_link"/>
+        <origin xyz="0.0 0.0 0.15" rpy="0 0 0"/>
+    </joint>
     <link name="base_link">
         <visual>
             <origin xyz="0 0 -0.15" rpy="0 0 1.57" />
             <geometry>
-                <mesh filename="package://limo_gazebo_sim/meshes/limo_base.dae" scale="1 1 1"/>
+                <mesh filename="package://limo_gazebo_sim/CAD/limo-model/limo_base.dae" scale="1 1 1"/>
             </geometry>
         </visual>
         <collision>
-            <!--origin xyz="0 0 -0.15" rpy="0 0 1.57" /-->
             <origin xyz="0 0 0" rpy="0 0 0" />
-          <geometry>
-              <box size="${base_x_size} ${base_y_size} ${base_z_size}"/>
-          </geometry>
+            <geometry>
+                <box size="${base_x_size} ${base_y_size} ${base_z_size}"/>
+            </geometry>
         </collision>
     </link>
@@ -52,4 +52,5 @@
         <child link="inertial_link" />
     </joint>
+    <!-- ================= 传感器装配 (包含 Gazebo 插件) ================= -->
     <xacro:limo_laser parent_prefix="base_link" frame_prefix="laser">
         <origin xyz="0.103 0 -0.034" rpy="0 0 0"/>
@@ -61,15 +62,87 @@
         <origin xyz="0.0 0 -0.1" rpy="0 0 0"/>
     </xacro:limo_imu>
+    <!-- ================= 四轮差速驱动轮系装配 ================= -->
+    <!-- 左前轮 -->
     <xacro:limo_wheel parent_prefix="base_link" wheel_prefix="front_left" reflect="1">
-        <origin xyz="${wheelbase/2} ${track/2} ${wheel_vertical_offset}" rpy="0 0  0" />
+        <origin xyz="${wheelbase/2} ${track/2} ${wheel_vertical_offset}" rpy="0 0 0" />
     </xacro:limo_wheel>
+    <xacro:limo_wheel_transmission wheel_prefix="front_left" />
+    <!-- 右前轮 -->
     <xacro:limo_wheel parent_prefix="base_link" wheel_prefix="front_right" reflect="-1">
         <origin xyz="${wheelbase/2} ${-track/2} ${wheel_vertical_offset}" rpy="${M_PI} 0 0" />
     </xacro:limo_wheel>
+    <xacro:limo_wheel_transmission wheel_prefix="front_right" />
+    <!-- 左后轮 -->
     <xacro:limo_wheel parent_prefix="base_link" wheel_prefix="rear_left" reflect="1">
         <origin xyz="${-wheelbase/2} ${track/2} ${wheel_vertical_offset}" rpy="0 0 0" />
     </xacro:limo_wheel>
+    <xacro:limo_wheel_transmission wheel_prefix="rear_left" />
+    <!-- 右后轮 -->
     <xacro:limo_wheel parent_prefix="base_link" wheel_prefix="rear_right" reflect="-1">
         <origin xyz="${-wheelbase/2} ${-track/2} ${wheel_vertical_offset}" rpy="${M_PI} 0 0" />
     </xacro:limo_wheel>
+    <xacro:limo_wheel_transmission wheel_prefix="rear_right" />
+    <!-- ================= Gazebo 仿真环境动力学与控制插件 ================= -->
+    <gazebo reference="front_left_wheel">
+        <mu1>10</mu1>
+        <mu2>10</mu2>
+        <kp>10000000.0</kp>
+        <kd>1.0</kd>
+        <minDepth>0.01</minDepth>
+        <fdir1>1 0 0</fdir1>
+        <maxContacts value="64"/>
+    </gazebo>
+    <gazebo reference="front_right_wheel">
+        <mu1>10</mu1>
+        <mu2>10</mu2>
+        <kp>10000000.0</kp>
+        <kd>1.0</kd>
+        <minDepth>0.01</minDepth>
+        <fdir1>1 0 0</fdir1>
+        <maxContacts value="64"/>
+    </gazebo>
+    <gazebo reference="rear_left_wheel">
+        <mu1>10</mu1>
+        <mu2>10</mu2>
+        <kp>10000000.0</kp>
+        <kd>1.0</kd>
+        <minDepth>0.01</minDepth>
+        <fdir1>1 0 0</fdir1>
+        <maxContacts value="64"/>
+    </gazebo>
+    <gazebo reference="rear_right_wheel">
+        <mu1>10</mu1>
+        <mu2>10</mu2>
+        <kp>10000000.0</kp>
+        <kd>1.0</kd>
+        <minDepth>0.01</minDepth>
+        <fdir1>1 0 0</fdir1>
+        <maxContacts value="64"/>
+    </gazebo>
+    <gazebo>
+        <!-- ros_control 控制器插件 -->
+        <plugin name="gazebo_ros_control" filename="libgazebo_ros_control.so">
+            <robotNamespace>$(arg robot_namespace)</robotNamespace>
+        </plugin>
+        <!-- 四轮差速滑移驱动插件 -->
+        <plugin name="four_diff_controller" filename="libgazebo_ros_skid_steer_drive.so">
+            <updateRate>100.0</updateRate>
+            <robotNamespace>$(arg robot_namespace)</robotNamespace>
+            <leftFrontJoint>front_left_wheel</leftFrontJoint>
+            <rightFrontJoint>front_right_wheel</rightFrontJoint>
+            <leftRearJoint>rear_left_wheel</leftRearJoint>
+            <rightRearJoint>rear_right_wheel</rightRearJoint>
+            <wheelSeparation>0.172</wheelSeparation>
+            <wheelDiameter>0.09</wheelDiameter>
+            <robotBaseFrame>base_footprint</robotBaseFrame>
+            <commandTopic>cmd_vel</commandTopic>
+            <torque>50</torque>
+            <broadcastTF>true</broadcastTF>
+            <odometryTopic>odom</odometryTopic>
+            <odometryFrame>odom</odometryFrame>
+            <covariance_x>0.000100</covariance_x>
+            <covariance_y>0.000100</covariance_y>
+            <covariance_yaw>0.010000</covariance_yaw>
+        </plugin>
+    </gazebo>
 </robot>

Commit message: 自适应阈值检测实现

File: src/limo_gazebo_sim/urdf/limo_ackerman.xacro (robot description, xacro)
@@ -7,14 +7,14 @@
     <!-- ================= 几何与物理参数定义 ================= -->
     <xacro:property name="M_PI" value="3.14159"/>
-    <xacro:property name="base_x_size" value="0.26" />
-    <xacro:property name="base_y_size" value="0.24" />
-    <xacro:property name="base_z_size" value="0.20" />
-    <xacro:property name="wheelbase" value="0.4"/>
-    <xacro:property name="track" value="0.28"/>
-    <xacro:property name="wheel_vertical_offset" value="-0.201996" />
+    <xacro:property name="base_x_size" value="0.286" />
+    <xacro:property name="base_y_size" value="0.264" />
+    <xacro:property name="base_z_size" value="0.220" />
+    <xacro:property name="wheelbase" value="0.44"/>
+    <xacro:property name="track" value="0.308"/>
+    <xacro:property name="wheel_vertical_offset" value="-0.222196" />
     <xacro:property name="base_mass" value="2.1557"/>
-    <xacro:property name="wheel_length" value="0.09" />
-    <xacro:property name="wheel_radius" value="0.09" />
-    <xacro:property name="wheel_scale" value="2 2 2" />
+    <xacro:property name="wheel_length" value="0.099" />
+    <xacro:property name="wheel_radius" value="0.099" />
+    <xacro:property name="wheel_scale" value="2.2 2.2 2.2" />
     <!-- ================= 底盘基准与车身 Link ================= -->
     <link name="base_footprint"/>
@@ -22,11 +22,11 @@
         <parent link="base_footprint"/>
         <child link="base_link"/>
-        <origin xyz="0.0 0.0 0.30" rpy="0 0 0"/>
+        <origin xyz="0.0 0.0 0.33" rpy="0 0 0"/>
     </joint>
     <link name="base_link">
         <visual>
-            <origin xyz="0 0 -0.30" rpy="0 0 1.57" />
+            <origin xyz="0 0 -0.33" rpy="0 0 1.57" />
             <geometry>
-                <mesh filename="package://limo_gazebo_sim/CAD/limo-model/limo_base.dae" scale="2 2 2"/>
+                <mesh filename="package://limo_gazebo_sim/CAD/limo-model/limo_base.dae" scale="2.2 2.2 2.2"/>
             </geometry>
         </visual>
@@ -54,11 +54,11 @@
     <!-- ================= 传感器装配 (包含 Gazebo 插件) ================= -->
     <xacro:limo_laser parent_prefix="base_link" frame_prefix="laser">
-        <origin xyz="0.206 0 -0.068" rpy="0 0 0"/>
+        <origin xyz="0.2266 0 -0.0748" rpy="0 0 0"/>
     </xacro:limo_laser>
     <xacro:limo_depth_camera parent_prefix="base_link" frame_prefix="depth_camera">
-        <origin xyz="0.168 0 0.06" rpy="0 0.2618 0"/>
+        <origin xyz="0.1848 0 0.066" rpy="0 0.2618 0"/>
     </xacro:limo_depth_camera>
     <xacro:limo_imu parent_prefix="base_link" frame_prefix="imu">
-        <origin xyz="0.0 0 -0.2" rpy="0 0 0"/>
+        <origin xyz="0.0 0 -0.22" rpy="0 0 0"/>
     </xacro:limo_imu>
     <!-- ================= 前轮转向机构装配 (转向铰链节 + 前轮) ================= -->
@@ -105,6 +105,6 @@
             <leftHingeJoint>left_steering_hinge_wheel</leftHingeJoint>
             <rightHingeJoint>right_steering_hinge_wheel</rightHingeJoint>
-            <wheelSeparation>0.344</wheelSeparation>
-            <wheelDiameter>0.18</wheelDiameter>
+            <wheelSeparation>0.3784</wheelSeparation>
+            <wheelDiameter>0.198</wheelDiameter>
             <wheelbase>${wheelbase}</wheelbase>
             <wheelTrack>${track}</wheelTrack>
